File: KiCad/new/PentaESPConverter.kicad_pcb (KiCad board)
At the start: 2 copper layers, 34.5 x 27.1 mm, 13 parts, among them J1 Conn_02x07_Odd_Even, J2 Conn_02x07_Odd_Even, J3 Conn_01x05, SW1 SW_Push, U1 AMS1117-3.3, U2 ESP32-WROOM-32

Commit message: added current PCB Design
Parts:
- moved U1 5.80 mm to (130.6, 107.7), turned to 270 degrees
- moved SW1 4.95 mm to (139.4, 112.2)
- moved D1 2.33 mm to (145.4, 112.3)
- moved R2 2.33 mm to (145.4, 109.2)
- moved C4 1.82 mm to (131.4, 100.5)
Connections:
- J2 pad 3: P36 -> JST3
- J2 pad 4: P35 -> JST2
- J2 pad 5: P34 -> JST4
- U2 pad 16: JST2 -> (no net)
- U2 pad 18: JST3 -> (no net)
- U2 pad 19: JST4 -> (no net)
- U2 pad 34: P34 -> JST4
- U2 pad 35: P35 -> JST2
- U2 pad 36: P36 -> JST3
Routing:
- net JST3: track 4.52 -> 31.9 mm
- net JST4: track 5.41 -> 29.5 mm
- net JST2: track 4.54 -> 27.8 mm
- net GND: track 30.1 -> 45.2 mm, vias 0 -> 1
- net P25: track 20.7 -> 7.77 mm
- net +5V: track 44.3 -> 57.0 mm
- net P36: track 6.65 -> 0.00 mm
- net P34: track 6.65 -> 0.00 mm
- net P35: track 3.66 -> 0.00 mm
- net P26: track 13.9 -> 12.0 mm
- net (no net): track 0.00 -> 0.77 mm
